File: hw/v02/noname.kicad_pcb (KiCad board)
At the start: 2 copper layers, 50.8 x 33 mm, 16 parts, among them J1 Conn_01x10_Female_Left, J2 Conn_01x10_Female_Right, SW1 EVQ-Q2Y03W, U1 MSP430G2553IPW28, U2 AT25640B-SSHL-T, U3 HDSM-283L, U4 HDSM-283L, U5 HDSM-283L, U6 HDSM-283L

Commit message: Tied eeprom 3 and 7 to VCC, board v04 RC
Connections:
- U2 pad 3: VCC -> Net-(U2-Pad3)
- U2 pad 7: VCC -> Net-(U2-Pad7)
Routing:
- net VCC: track 52.6 -> 42.2 mm, vias 2 -> 0
Other:
- board text added: "v03"
- board text removed: "v04"
Changed lines of the file:
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@@
-(kicad_pcb (version 20171130) (host pcbnew 5.1.5-52549c5~86~ubuntu18.04.1)
+(kicad_pcb (version 20171130) (host pcbnew 5.1.5-52549c5~84~ubuntu18.04.1)
   (general
     (thickness 1.6)
     (drawings 11)
-    (tracks 413)
+    (tracks 403)
     (zones 0)
     (modules 16)
-    (nets 49)
+    (nets 51)
   )
   (page A4)
   (layers
     (0 F.Cu signal)
-    (31 B.Cu signal)
-    (32 B.Adhes user)
-    (33 F.Adhes user)
-    (34 B.Paste user)
-    (35 F.Paste user)
-    (36 B.SilkS user)
-    (37 F.SilkS user)
-    (38 B.Mask user)
-    (39 F.Mask user)
-    (40 Dwgs.User user)
-    (41 Cmts.User user)
-    (42 Eco1.User user)
-    (43 Eco2.User user)
-    (44 Edge.Cuts user)
-    (45 Margin user)
+    (31 B.Cu signal hide)
+    (32 B.Adhes user hide)
+    (33 F.Adhes user hide)
+    (34 B.Paste user hide)
+    (35 F.Paste user hide)
+    (36 B.SilkS user hide)
+    (37 F.SilkS user hide)
+    (38 B.Mask user hide)
+    (39 F.Mask user hide)
+    (40 Dwgs.User user hide)
+    (41 Cmts.User user hide)
+    (42 Eco1.User user hide)
+    (43 Eco2.User user hide)
+    (44 Edge.Cuts user hide)
+    (45 Margin user hide)
     (46 B.CrtYd user hide)
     (47 F.CrtYd user hide)
@@
     (solder_mask_min_width 0.25)
     (aux_axis_origin 0 0)
-    (visible_elements FFFFFF7F)
+    (visible_elements FFF9E71F)
     (pcbplotparams
       (layerselection 0x010fc_ffffffff)
@@
   (net 35 /DIG_2)
   (net 36 /SCK)
-  (net 37 "Net-(U3-Pad9)")
-  (net 38 "Net-(U3-Pad7)")
-  (net 39 "Net-(U3-Pad2)")
-  (net 40 "Net-(U4-Pad9)")
-  (net 41 "Net-(U4-Pad7)")
-  (net 42 "Net-(U4-Pad2)")
-  (net 43 "Net-(U5-Pad9)")
-  (net 44 "Net-(U5-Pad7)")
-  (net 45 "Net-(U5-Pad2)")
-  (net 46 "Net-(U6-Pad9)")
-  (net 47 "Net-(U6-Pad7)")
-  (net 48 "Net-(U6-Pad2)")
+  (net 37 "Net-(U2-Pad7)")
+  (net 38 "Net-(U2-Pad3)")
+  (net 39 "Net-(U3-Pad9)")
+  (net 40 "Net-(U3-Pad7)")
+  (net 41 "Net-(U3-Pad2)")
+  (net 42 "Net-(U4-Pad9)")
+  (net 43 "Net-(U4-Pad7)")
+  (net 44 "Net-(U4-Pad2)")
+  (net 45 "Net-(U5-Pad9)")
+  (net 46 "Net-(U5-Pad7)")
+  (net 47 "Net-(U5-Pad2)")
+  (net 48 "Net-(U6-Pad9)")
+  (net 49 "Net-(U6-Pad7)")
+  (net 50 "Net-(U6-Pad2)")
   (net_class Default "This is the default net class."
     (clearance 0.2)
@@
     (add_net "Net-(J2-PadP2.6)")
     (add_net "Net-(J2-PadP2.7)")
+    (add_net "Net-(U2-Pad3)")
+    (add_net "Net-(U2-Pad7)")
     (add_net "Net-(U3-Pad2)")
     (add_net "Net-(U3-Pad7)")
@@
       (net 1 VCC))
     (pad 7 smd roundrect (at 2.475 -0.635 90) (size 1.95 0.6) (layers F.Cu F.Paste F.Mask) (roundrect_rratio 0.25)
-      (net 1 VCC))
+      (net 37 "Net-(U2-Pad7)"))
     (pad 6 smd roundrect (at 2.475 0.635 90) (size 1.95 0.6) (layers F.Cu F.Paste F.Mask) (roundrect_rratio 0.25)
       (net 36 /SCK))
@@
       (net 2 GND))
     (pad 3 smd roundrect (at -2.475 0.635 90) (size 1.95 0.6) (layers F.Cu F.Paste F.Mask) (roundrect_rratio 0.25)
-      (net 1 VCC))
+      (net 38 "Net-(U2-Pad3)"))
     (pad 2 smd roundrect (at -2.475 -0.635 90) (size 1.95 0.6) (layers F.Cu F.Paste F.Mask) (roundrect_rratio 0.25)
       (net 25 /SOMI))
@@
       (net 29 /SEG_D))
     (pad 9 smd rect (at 0.635 5.4) (size 0.8 3) (layers F.Cu F.Paste F.Mask)
-      (net 46 "Net-(U6-Pad9)"))
+      (net 48 "Net-(U6-Pad9)"))
     (pad 8 smd rect (at 1.905 5.4) (size 0.8 3) (layers F.Cu F.Paste F.Mask)
       (net 31 /SEG_C))
     (pad 7 smd rect (at 3.175 5.4) (size 0.8 3) (layers F.Cu F.Paste F.Mask)
-      (net 47 "Net-(U6-Pad7)"))
+      (net 49 "Net-(U6-Pad7)"))
     (pad 6 smd rect (at 3.175 -5.4) (size 0.8 3) (layers F.Cu F.Paste F.Mask)
       (net 32 /SEG_B))
@@
       (net 27 /SEG_F))
     (pad 2 smd rect (at -1.905 -5.4) (size 0.8 3) (layers F.Cu F.Paste F.Mask)
-      (net 48 "Net-(U6-Pad2)"))
+      (net 50 "Net-(U6-Pad2)"))
     (pad 1 smd rect (at -3.175 -5.4) (size 0.8 3) (layers F.Cu F.Paste F.Mask)
       (net 23 /SEG_G))
@@
       (net 29 /SEG_D))
     (pad 9 smd rect (at 0.635 5.4) (size 0.8 3) (layers F.Cu F.Paste F.Mask)
-      (net 43 "Net-(U5-Pad9)"))
+      (net 45 "Net-(U5-Pad9)"))
     (pad 8 smd rect (at 1.905 5.4) (size 0.8 3) (layers F.Cu F.Paste F.Mask)
       (net 31 /SEG_C))
     (pad 7 smd rect (at 3.175 5.4) (size 0.8 3) (layers F.Cu F.Paste F.Mask)
-      (net 44 "Net-(U5-Pad7)"))
+      (net 46 "Net-(U5-Pad7)"))
     (pad 6 smd rect (at 3.175 -5.4) (size 0.8 3) (layers F.Cu F.Paste F.Mask)
       (net 32 /SEG_B))
@@
       (net 27 /SEG_F))
     (pad 2 smd rect (at -1.905 -5.4) (size 0.8 3) (layers F.Cu F.Paste F.Mask)
-      (net 45 "Net-(U5-Pad2)"))
+      (net 47 "Net-(U5-Pad2)"))
     (pad 1 smd rect (at -3.175 -5.4) (size 0.8 3) (layers F.Cu F.Paste F.Mask)
       (net 23 /SEG_G))
@@
       (net 29 /SEG_D))
     (pad 9 smd rect (at 0.635 5.4) (size 0.8 3) (layers F.Cu F.Paste F.Mask)
-      (net 40 "Net-(U4-Pad9)"))
+      (net 42 "Net-(U4-Pad9)"))
     (pad 8 smd rect (at 1.905 5.4) (size 0.8 3) (layers F.Cu F.Paste F.Mask)
       (net 31 /SEG_C))
     (pad 7 smd rect (at 3.175 5.4) (size 0.8 3) (layers F.Cu F.Paste F.Mask)
-      (net 41 "Net-(U4-Pad7)"))
+      (net 43 "Net-(U4-Pad7)"))
     (pad 6 smd rect (at 3.175 -5.4) (size 0.8 3) (layers F.Cu F.Paste F.Mask)
       (net 32 /SEG_B))
@@
       (net 27 /SEG_F))
     (pad 2 smd rect (at -1.905 -5.4) (size 0.8 3) (layers F.Cu F.Paste F.Mask)
-      (net 42 "Net-(U4-Pad2)"))
+      (net 44 "Net-(U4-Pad2)"))
     (pad 1 smd rect (at -3.175 -5.4) (size 0.8 3) (layers F.Cu F.Paste F.Mask)
       (net 23 /SEG_G))
@@
       (net 29 /SEG_D))
     (pad 9 smd rect (at 0.635 5.4) (size 0.8 3) (layers F.Cu F.Paste F.Mask)
-      (net 37 "Net-(U3-Pad9)"))
+      (net 39 "Net-(U3-Pad9)"))
     (pad 8 smd rect (at 1.905 5.4) (size 0.8 3) (layers F.Cu F.Paste F.Mask)
       (net 31 /SEG_C))
     (pad 7 smd rect (at 3.175 5.4) (size 0.8 3) (layers F.Cu F.Paste F.Mask)
-      (net 38 "Net-(U3-Pad7)"))
+      (net 40 "Net-(U3-Pad7)"))
     (pad 6 smd rect (at 3.175 -5.4) (size 0.8 3) (layers F.Cu F.Paste F.Mask)
       (net 32 /SEG_B))
@@
       (net 27 /SEG_F))
     (pad 2 smd rect (at -1.905 -5.4) (size 0.8 3) (layers F.Cu F.Paste F.Mask)
-      (net 39 "Net-(U3-Pad2)"))
+      (net 41 "Net-(U3-Pad2)"))
     (pad 1 smd rect (at -3.175 -5.4) (size 0.8 3) (layers F.Cu F.Paste F.Mask)
       (net 23 /SEG_G))
@@
   (gr_arc (start 125.73 100.33) (end 124.46 100.33) (angle -90) (layer Edge.Cuts) (width 0.05))
   (gr_arc (start 125.73 69.85) (end 125.73 68.58) (angle -90) (layer Edge.Cuts) (width 0.05))
-  (gr_text v04 (at 125.73 70.485) (layer F.SilkS)
+  (gr_text v03 (at 125.73 70.485) (layer F.SilkS)
     (effects (font (size 1 1) (thickness 0.15)) (justify left))
   )
@@
   (segment (start 149.225 73.025) (end 153.67 73.025) (width 0.5) (layer F.Cu) (net 1))
   (segment (start 157.48 71.12) (end 157.48 73.4075) (width 0.4) (layer F.Cu) (net 1))
-  (segment (start 158.75 73.4075) (end 157.48 73.4075) (width 0.25) (layer F.Cu) (net 1))
-  (via (at 160.037331 76.266699) (size 0.8) (drill 0.4) (layers F.Cu B.Cu) (net 1))
-  (segment (start 160.02 78.3575) (end 160.02 76.28403) (width 0.25) (layer F.Cu) (net 1))
-  (segment (start 160.02 76.28403) (end 160.037331 76.266699) (width 0.25) (layer F.Cu) (net 1))
-  (via (at 156.21 73.66) (size 0.8) (drill 0.4) (layers F.Cu B.Cu) (net 1))
-  (segment (start 157.48 73.4075) (end 156.4625 73.4075) (width 0.25) (layer F.Cu) (net 1))
-  (segment (start 156.4625 73.4075) (end 156.21 73.66) (width 0.25) (layer F.Cu) (net 1))
-  (segment (start 156.21 73.66) (end 156.21 74.93) (width 0.25) (layer B.Cu) (net 1))
-  (segment (start 157.546699 76.266699) (end 160.037331 76.266699) (width 0.25) (layer B.Cu) (net 1))
-  (segment (start 156.21 74.93) (end 157.546699 76.266699) (width 0.25) (layer B.Cu) (net 1))
   (segment (start 143.51 78.105) (end 143.525 78.12) (width 0.25) (layer B.Cu) (net 2))
   (segment (start 156.21 78.105) (end 156.195 78.12) (width 0.25) (layer B.Cu) (net 2))
